Commit message: added launch file

File: urdf/hokuyo_laser.urdf.xacro (robot description, xacro)
@@ -3,15 +3,5 @@
   <!-- Include the hokuyo_ust10 xacro -->
   <xacro:include filename="$(find urg_node)/urdf/hokuyo_ust10.urdf.xacro"/>
-  <!-- Define material -->
-  <material name="dark_grey">
-    <color rgba="0.3 0.3 0.3 1"/>
-  </material>
   <link name="world"/>
-  <!-- <link name="base_link"/>
-  <joint name="world_to_base" type="fixed">
-    <origin rpy="0 0 0" xyz="0 0 0"/>
-    <parent link="world"/>
-    <child link="base_link"/>
-  </joint> -->
   <!-- Use the hokuyo_ust10_mount macro -->
   <xacro:hokuyo_ust10_mount prefix="hokuyo" topic="scan" parent_link="world">

File: urdf/hokuyo_ust10.urdf.xacro (robot description, xacro)
@@ -1,4 +1,5 @@
 <?xml version="1.0"?>
 <robot name="hokuyo_ust10" xmlns:xacro="http://ros.org/wiki/xacro">
+<xacro:include filename="$(find urg_node)/urdf/materials.urdf.xacro"/>
   <xacro:macro name="hokuyo_ust10_mount" params="prefix topic parent_link min_angle:=-2.35619 max_angle:=2.35619 *origin">
     <xacro:macro name="hokuyo_ust10" params="frame:=laser topic:=scan sample_size:=720 update_rate:=50
