Commit message: fixed non-working codes

File: urdf/hokuyo_ust10.urdf.xacro (robot description, xacro)
@@ -1,4 +1,4 @@
 <?xml version="1.0"?>
-<robot xmlns:xacro="http://ros.org/wiki/xacro">
+<robot name="hokuyo_ust10" xmlns:xacro="http://ros.org/wiki/xacro">
   <xacro:macro name="hokuyo_ust10_mount" params="prefix topic parent_link min_angle:=-2.35619 max_angle:=2.35619 *origin">
     <xacro:macro name="hokuyo_ust10" params="frame:=laser topic:=scan sample_size:=720 update_rate:=50
@@ -76,3 +76,9 @@
     </gazebo>
   </xacro:macro>
+  <!-- Create a base_link and use the macro -->
+  <!-- <link name="base_link"/> -->
+  <!-- Example usage of the macro -->
+  <!-- <xacro:hokuyo_ust10_mount prefix="laser" topic="scan" parent_link="base_link">
+    <origin xyz="0 0 0" rpy="0 0 0"/>
+  </xacro:hokuyo_ust10_mount> -->
 </robot>

Commit message: fixed mesh import

File: urdf/hokuyo_ust10.urdf.xacro (robot description, xacro)
@@ -62,5 +62,5 @@
         <geometry>
           <!-- Origin of this mesh is the base of the bracket. -->
-          <mesh filename="package://urg_node/meshes/hokuyo_ust10.stl" />
+          <mesh filename="file://$(find urg_node)/meshes/hokuyo_ust10.stl"/>
         </geometry>
         <material name="dark_grey" />

Commit message: reduced laser resolution for matlab compatibility

File: urdf/hokuyo_ust10.urdf.xacro (robot description, xacro)
@@ -3,5 +3,5 @@
 <xacro:include filename="$(find urg_node)/urdf/materials.urdf.xacro"/>
   <xacro:macro name="hokuyo_ust10_mount" params="prefix topic parent_link min_angle:=-2.35619 max_angle:=2.35619 *origin">
-    <xacro:macro name="hokuyo_ust10" params="frame:=laser topic:=scan sample_size:=720 update_rate:=50
+    <xacro:macro name="hokuyo_ust10" params="frame:=laser topic:=scan sample_size:=120 update_rate:=50
                min_angle:=${min_angle} max_angle:=${max_angle} min_range:=0.1 max_range:=30.0 robot_namespace:=/">
       <link name="${frame}">

Commit message: reduced lidar publishing frequency

File: urdf/hokuyo_ust10.urdf.xacro (robot description, xacro)
@@ -3,5 +3,5 @@
 <xacro:include filename="$(find urg_node)/urdf/materials.urdf.xacro"/>
   <xacro:macro name="hokuyo_ust10_mount" params="prefix topic parent_link min_angle:=-2.35619 max_angle:=2.35619 *origin">
-    <xacro:macro name="hokuyo_ust10" params="frame:=laser topic:=scan sample_size:=120 update_rate:=50
+    <xacro:macro name="hokuyo_ust10" params="frame:=laser topic:=scan sample_size:=120 update_rate:=10
                min_angle:=${min_angle} max_angle:=${max_angle} min_range:=0.1 max_range:=30.0 robot_namespace:=/">
       <link name="${frame}">
